Commit message: barco funciona no gazebo controlador por comando ps5

File: ats_description/urdf/example_component_config.xacro (robot description, xacro)
@@ -7,3 +7,3 @@
       <xacro:wamv_imu name="imu_wamv" x="0.3" y="-0.2" z="1.3" R="0.0" P="0.0" Y="0.0" />
   </xacro:macro>
-</robot>
+</robot>\

File: ats_description/urdf/wamv_target.urdf.xacro (robot description, xacro)
@@ -336,8 +336,9 @@
   <joint name="wamv/left_chassis_engine_joint" type="revolute">
     <axis xyz="0 0 1"/>
-    <limit effort="10" lower="-3.141592653589793" upper="3.141592653589793" velocity="10"/>
+    <limit effort="1000" lower="-3.141592653589793" upper="3.141592653589793" velocity="10"/>
     <origin rpy="0.0 0.0 0.0" xyz="-2.373776 1.027135 0.318237"/>
     <parent link="wamv/base_link"/>
     <child link="wamv/left_engine_link"/>
+    <dynamics damping="10.0" friction="10.0"/>
   </joint>
   <joint name="wamv/left_engine_propeller_joint" type="continuous">
@@ -391,8 +392,9 @@
   <joint name="wamv/right_chassis_engine_joint" type="revolute">
     <axis xyz="0 0 1"/>
-    <limit effort="10" lower="-3.141592653589793" upper="3.141592653589793" velocity="10"/>
+    <limit effort="1000" lower="-3.141592653589793" upper="3.141592653589793" velocity="10"/>
     <origin rpy="0.0 0.0 0.0" xyz="-2.373776 -1.027135 0.318237"/>
     <parent link="wamv/base_link"/>
     <child link="wamv/right_engine_link"/>
+    <dynamics damping="10.0" friction="10.0"/>
   </joint>
   <joint name="wamv/right_engine_propeller_joint" type="continuous">
@@ -670,48 +672,3 @@
     </sensor>
   </gazebo>
-  <link name="wamv/cpu_cases_link">
-    <visual>
-      <origin rpy="0 0 0" xyz="0.073 0 -1.53"/>
-      <geometry>
-        <mesh filename="package://vrx_gazebo/models/cpu_cases/mesh/cpu_cases.dae"/>
-      </geometry>
-    </visual>
-    <collision name="cpu_case_1_collision">
-      <origin rpy="0 0 0" xyz="0.185 0 0"/>
-      <geometry>
-        <box size="0.595 0.83 0.47"/>
-      </geometry>
-    </collision>
-    <collision name="cpu_case_2_collision">
-      <origin rpy="0 0 0" xyz="-0.3 0 -0.092"/>
-      <geometry>
-        <box size="0.375 0.64 0.28"/>
-      </geometry>
-    </collision>
-    <inertial>
-      <mass value="20"/>
-      <inertia ixx="1.51633333333333" ixy="0" ixz="0" iyy="1.93633333333333" iyz="0" izz="2.71633333333333"/>
-    </inertial>
-  </link>
-  <joint name="wamv/chasis_cpu_cases_joint" type="fixed">
-    <origin rpy="0 0 0" xyz="-0.15 0 1.53"/>
-    <parent link="wamv/base_link"/>
-    <child link="wamv/cpu_cases_link"/>
-  </joint>
-  <gazebo reference="wamv/cpu_cases_link">
-    <visual>
-      <material>
-        <diffuse>1.0 1.0 1.0</diffuse>
-        <specular>1.0 1.0 1.0</specular>
-        <pbr>
-          <metal>
-            <albedo_map>model://vrx_gazebo/models/cpu_cases/mesh/cpu_cases_Albedo.png</albedo_map>
-            <normal_map>model://vrx_gazebo/models/cpu_cases/mesh/cpu_cases_Normal.png</normal_map>
-            <roughness_map>model://vrx_gazebo/models/cpu_cases/mesh/cpu_cases_Roughness.png</roughness_map>
-            <metalness_map>model://vrx_gazebo/models/cpu_cases/mesh/cpu_cases_Metalness.png</metalness_map>
-          </metal>
-        </pbr>
-      </material>
-    </visual>
-  </gazebo>
 </robot>
