Commit message: added a script to generate the tether sdf, and conected the tether to the wamv

File: ats_description/urdf/wamv_target.urdf.xacro (robot description, xacro)
@@ -678,3 +678,21 @@
     </sensor>
   </gazebo>
+  <link name="wamv/tether_anchor">
+    <!-- Visual removido para estética -->
+    <collision name="wamv/tether_anchor_collision">
+      <geometry><sphere radius="0.01"/></geometry>
+    </collision>
+    <inertial>
+      <mass value="0.1"/>
+      <inertia ixx="0.0001" ixy="0" ixz="0" iyy="0.0001" iyz="0" izz="0.0001"/>
+    </inertial>
+  </link>
+  <joint name="wamv/tether_anchor_joint" type="fixed">
+    <origin rpy="0 0 0" xyz="-0.70 0.0 1.3"/>
+    <parent link="wamv/base_link"/>
+    <child link="wamv/tether_anchor"/>
+  </joint>
+  <gazebo reference="wamv/tether_anchor_joint">
+    <preserveFixedJoint>true</preserveFixedJoint>
+  </gazebo>
 </robot>

Commit message: make the tether part of the boat, and activate self collision

File: ats_description/urdf/wamv_target.urdf.xacro (robot description, xacro)
@@ -5,5 +5,5 @@
 <!-- =================================================================================== -->
 <!-- Basic WAM-V with gazebo plugins for dynamics -->
-<robot name="WAM-V">
+<robot name="WAM-V" xmlns:xacro="http://ros.org/wiki/xacro">
   <link name="wamv/left_battery_link">
     <visual>
@@ -696,3 +696,25 @@
     <preserveFixedJoint>true</preserveFixedJoint>
   </gazebo>
+  <!-- Ativar colisões internas para que o tether (e outras partes móveis) colidam com o barco -->
+  <gazebo>
+    <self_collide>true</self_collide>
+  </gazebo>
+  <!-- Inclusão Condicional do Tether como Modelo Aninhado -->
+  <xacro:arg name="has_tether" default="false"/>
+  <xacro:if value="$(arg has_tether)">
+    <gazebo>
+      <include>
+        <uri>model://tether</uri>
+        <!-- A pose do tether é relativa à âncora, logo 0 0 0 -->
+        <pose>-0.70 0.0 1.3 0 0 0</pose>
+      </include>
+      <!-- Usar uma junta universal ou ball para o ponto de fixação para garantir flexibilidade -->
+      <joint name="tether_to_boat_joint" type="universal">
+        <parent>wamv/tether_anchor</parent>
+        <child>tether::link_base</child>
+        <axis><xyz>1 0 0</xyz><dynamics><damping>0.1</damping></dynamics></axis>
+        <axis2><xyz>0 1 0</xyz><dynamics><damping>0.1</damping></dynamics></axis2>
+      </joint>
+    </gazebo>
+  </xacro:if>
 </robot>

Commit message: change wamv model from xacro to fixed sdf

File: ats_description/urdf/wamv_target.urdf.xacro (robot description, xacro)
@@ -678,43 +678,3 @@
     </sensor>
   </gazebo>
-  <link name="wamv/tether_anchor">
-    <!-- Visual removido para estética -->
-    <collision name="wamv/tether_anchor_collision">
-      <geometry><sphere radius="0.01"/></geometry>
-    </collision>
-    <inertial>
-      <mass value="0.1"/>
-      <inertia ixx="0.0001" ixy="0" ixz="0" iyy="0.0001" iyz="0" izz="0.0001"/>
-    </inertial>
-  </link>
-  <joint name="wamv/tether_anchor_joint" type="fixed">
-    <origin rpy="0 0 0" xyz="-0.70 0.0 1.3"/>
-    <parent link="wamv/base_link"/>
-    <child link="wamv/tether_anchor"/>
-  </joint>
-  <gazebo reference="wamv/tether_anchor_joint">
-    <preserveFixedJoint>true</preserveFixedJoint>
-  </gazebo>
-  <!-- Ativar colisões internas para que o tether (e outras partes móveis) colidam com o barco -->
-  <gazebo>
-    <self_collide>true</self_collide>
-  </gazebo>
-  <!-- Inclusão Condicional do Tether como Modelo Aninhado -->
-  <xacro:arg name="has_tether" default="false"/>
-  <xacro:if value="$(arg has_tether)">
-    <gazebo>
-      <include>
-        <uri>model://tether</uri>
-        <!-- A pose do tether é relativa à âncora, logo 0 0 0 -->
-        <pose>-0.70 0.0 1.3 0 0 0</pose>
-      </include>
-      <!-- Usar uma junta universal ou ball para o ponto de fixação para garantir flexibilidade -->
-      <joint name="tether_to_boat_joint" type="universal">
-        <parent>wamv/tether_anchor</parent>
-        <child>tether::link_base</child>
-        <axis><xyz>1 0 0</xyz><dynamics><damping>0.1</damping></dynamics></axis>
-        <axis2><xyz>0 1 0</xyz><dynamics><damping>0.1</damping></dynamics></axis2>
-      </joint>
-    </gazebo>
-  </xacro:if>
 </robot>
