Commit message: changed package names

File: simulation/description/urdf/wamv.urdf (robot description, URDF)
Before this commit: robot wamv, 1 links, 0 joints
Links:
- link boat/base_link: geometry visual mesh filename=package://description/models/wamv/meshes/WAM-V-Base.dae

File: simulation/description/urdf/x500.urdf (robot description, URDF)
Before this commit: robot x500, 1 links, 0 joints
Links:
- link drone/base_link: geometry visual mesh filename=package://description/models/x500_base/meshes/NXP-HGD-CF.dae
