Commit message: simulation: landing pad on the WAM-V above the tether winch
Flat plate with walls at 45 deg that centre the landing gear, added to the
SDF (collision and visual) and to the URDF (visual). The UAV now spawns on
the pad. The URDF hull mesh gets the same offset from base_link as in the SDF.

Co-Authored-By: Claude Opus 5.5 <noreply@anthropic.com>
Claude-Session: https://claude.ai/code/session_01QNxivjCqsxdeckdqAgRe9o

File: simulation/description/urdf/wamv.urdf (robot description, URDF)
Before this commit: robot wamv, 1 links, 0 joints
Links:
- link boat/base_link: geometry visual box size=0.1414 0.6000 0.0100; visual box size=0.1414 0.6000 0.0100

Commit message: description: thrusters, rotors and sea level for visualisation
WAM-V thrusters and x500 motors and propellers in the URDFs (propellers as
COLLADA in the rotor frame), and a mean sea level plane.

Co-Authored-By: Claude Opus 5.5 <noreply@anthropic.com>
Claude-Session: https://claude.ai/code/session_01QNxivjCqsxdeckdqAgRe9o

File: simulation/description/urdf/wamv.urdf (robot description, URDF)
Before this commit: robot wamv, 1 links, 0 joints
Links:
- link boat/base_link: geometry visual box size=0.1414 0.6000 0.0100; visual box size=0.1414 0.6000 0.0100

File: simulation/description/urdf/x500.urdf (robot description, URDF)
Before this commit: robot x500, 1 links, 0 joints
Links:
- link drone/base_link: geometry visual mesh filename=package://description/models/x500_base/meshes/1345_prop_ccw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; visual mesh filename=package://description/models/x500_base/meshes/1345_prop_ccw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
